File: PCB/PrimaryBoard-ASA/PrimaryBoard-ASA.kicad_sch (KiCad schematic)
At the start: 15 parts, among them J1 boardToBoard-ASA(8PIN), J2 boardToBoard-SPI, J4 ANT_Connector, J5 Pad, U1 BMP280, U2 ICM20948, U3 ESP32-S3-SUPERMIINI, U4 TuboPitot, U5 RF95W, U6 GY-ADS1115

Commit message: add midia
Parts:
- J3: value ~ -> (none)
Other:
- title: (none) -> VANT-PCBinferior
- moved on the sheet: C1, J4, J5, JP1, JP2, U5
